File: riaa.kicad_pcb (KiCad board)
At the start: 2 copper layers, 74 parts, among them J1 IN, J2 POWER, J3 IN, J4 OUT, J5 OUT

Commit message: Fix resistors
Parts:
- R13, R14, R23, R24, R29, R30, R31, R32, R33, R34, R35, R36, VT1, VT2, VT3, VT4: moved to B.Cu
- R19, R20, R21, R22: value 510 -> 1.2k; footprint Resistors_ThroughHole:R_Axial_DIN0918_L18.0mm_D9.0mm_P22.86mm_Horizontal -> Resistors_ThroughHole:R_Axial_DIN0617_L17.0mm_D6.0mm_P20.32mm_Horizontal
- moved R19 181.0 mm to (222.4, 95.0), turned to 90 degrees
- moved R20 167.2 mm to (212.2, 41.5), turned to 270 degrees
- moved R21 155.6 mm to (180.9, 122.7)
- moved R14 123.8 mm to (174.0, 68.8), turned to 270 degrees
- moved R28 117.1 mm to (190.4, 99.0)
- moved R23 113.3 mm to (186.8, 79.0)
- moved D4 112.0 mm to (180.0, 92.4), turned to 270 degrees
- moved R30 111.3 mm to (199.0, 36.6)
- moved R17 108.7 mm to (182.1, 57.1), turned to 180 degrees
- moved D3 102.2 mm to (180.1, 77.5), turned to 90 degrees
- moved VT1 102.0 mm to (192.8, 79.2)
- moved VT2 99.7 mm to (198.7, 56.5)
- moved R13 92.5 mm to (173.6, 91.0), turned to 270 degrees
- moved D2 92.0 mm to (173.4, 77.8), turned to 90 degrees
- moved VT4 90.5 mm to (253.7, 48.5)
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Routing:
- net GNDA: track 150.2 -> 175.8 mm
- net Net-(C3-Pad1): track 13.6 -> 25.8 mm
- net Net-(C4-Pad1): track 23.8 -> 35.9 mm
- net Net-(C19-Pad1): track 21.4 -> 24.8 mm
- net Net-(C20-Pad1): track 23.4 -> 26.4 mm
- net Net-(C10-Pad1): track 10.3 -> 11.6 mm

Commit message: Fix PCB
Parts:
- removed C13, C14: 2.2, Capacitors_ThroughHole:CP_Radial_D6.3mm_P2.50mm
- removed C17, C18: 0.1, Capacitors_ThroughHole:C_Rect_L9.0mm_W4.9mm_P7.50mm_MKT
- moved R22 146.4 mm to (212.4, 90.2), turned to 90 degrees
- moved J2 130.0 mm to (220.0, 77.9)
- moved R36 121.5 mm to (212.4, 80.0), turned to 90 degrees
- moved C16 109.1 mm to (218.8, 67.1), turned to 270 degrees
- moved R31 106.4 mm to (194.4, 63.1), turned to 270 degrees
- moved R35 105.7 mm to (209.0, 97.8), turned to 90 degrees
- moved R34 97.3 mm to (204.4, 95.6)
- moved R33 91.7 mm to (200.3, 91.9), turned to 180 degrees
- moved R24 88.0 mm to (194.0, 101.8)
- moved R29 82.4 mm to (205.2, 78.2), turned to 90 degrees
- moved R26 80.6 mm to (191.8, 105.0), turned to 90 degrees
- moved C12 78.6 mm to (214.2, 60.7), turned to 270 degrees
- moved VT4 62.9 mm to (208.8, 92.6), turned to 90 degrees
- moved VT3 62.4 mm to (198.0, 88.8), turned to 90 degrees
- moved C15 52.4 mm to (218.8, 93.7), turned to 90 degrees
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Connections:
- DA2 pad 1: (no net) -> Net-(DA2-Pad1)
- DA2 pad 5: Net-(DA2-Pad5) -> Net-(DA2-Pad1)
- DA3 pad 1: (no net) -> Net-(DA3-Pad1)
- DA3 pad 5: Net-(DA3-Pad5) -> Net-(DA3-Pad1)
- R27 pad 1: Net-(DA2-Pad8) -> Net-(DA2-Pad1)
- R27 pad 3: Net-(DA2-Pad5) -> Net-(DA2-Pad8)
- R28 pad 1: Net-(DA3-Pad8) -> Net-(DA3-Pad1)
- R28 pad 3: Net-(DA3-Pad5) -> Net-(DA3-Pad8)
Routing:
- net GNDA: track 175.8 -> 381.6 mm
- net VCC: track 0.00 -> 105.8 mm
- net VEE: track 0.00 -> 84.1 mm
- net Net-(C22-Pad2): track 0.00 -> 75.6 mm
- net Net-(DA2-Pad1): track 0.00 -> 58.7 mm
- net Net-(DA3-Pad6): track 0.00 -> 58.3 mm
- net Net-(DA2-Pad6): track 0.00 -> 56.3 mm
- net Net-(C21-Pad1): track 0.00 -> 51.2 mm
- net Net-(C22-Pad1): track 0.00 -> 50.4 mm
- net Net-(DA3-Pad1): track 0.00 -> 45.4 mm, vias 0 -> 2
- net Net-(C21-Pad2): track 0.00 -> 30.0 mm
- net Net-(DA3-Pad2): track 0.00 -> 21.1 mm
- net Net-(R20-Pad1): track 0.00 -> 20.9 mm
- net Net-(DA2-Pad8): track 0.00 -> 19.0 mm
- net Net-(DA2-Pad2): track 0.00 -> 19.0 mm
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- added copper zone on B.Cu, net GNDA
Other:
- board outline added: 95.5 x 61.5 mm

Commit message: Fix PCB
Parts:
- moved R33 12.1 mm to (211.6, 96.2), turned to 90 degrees
- moved VT4 9.55 mm to (202.1, 85.8), turned to 0 degrees
- moved R35 9.47 mm to (200.0, 94.8)
- moved R23 8.18 mm to (208.7, 63.0)
- moved R34 6.85 mm to (197.6, 94.8), turned to 270 degrees
- moved R30 4.99 mm to (198.7, 68.9)
- moved R28 4.05 mm to (203.4, 98.6), turned to 0 degrees
- moved R27 3.97 mm to (203.5, 61.3), turned to 180 degrees
- moved VT3 3.73 mm to (195.7, 85.9)
- moved VT1 2.50 mm to (206.0, 66.5)
- moved R24 2.09 mm to (194.6, 99.8)
- moved R36 2.00 mm to (210.4, 80.0)
Connections:
- R27 pad 1: Net-(DA2-Pad1) -> Net-(DA2-Pad8)
- R27 pad 3: Net-(DA2-Pad8) -> Net-(DA2-Pad1)
- R28 pad 1: Net-(DA3-Pad1) -> Net-(DA3-Pad8)
- R28 pad 3: Net-(DA3-Pad8) -> Net-(DA3-Pad1)
Routing:
- net GNDA: track 381.6 -> 563.5 mm
- net Net-(DA2-Pad1): track 58.7 -> 39.4 mm
- net Net-(C22-Pad2): track 75.6 -> 59.6 mm
- net Net-(R35-Pad2): track 18.8 -> 34.7 mm
- net Net-(R33-Pad2): track 8.60 -> 22.7 mm
- net Net-(R22-Pad1): track 4.62 -> 16.5 mm
- net (no net): track 12.2 -> 1.87 mm
- net Net-(C21-Pad1): track 51.2 -> 60.7 mm
- net Net-(DA3-Pad6): track 58.3 -> 66.7 mm
- net Net-(C22-Pad1): track 50.4 -> 56.5 mm
- net Net-(DA2-Pad8): track 19.0 -> 24.4 mm
- net VEE: track 84.1 -> 78.9 mm
- net Net-(DA2-Pad6): track 56.3 -> 60.9 mm
- net Net-(R24-Pad2): track 5.27 -> 7.70 mm
- net Net-(R23-Pad2): track 2.92 -> 5.32 mm
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
Commit message: Fix PCB
Parts:
- moved D4 0.25 mm to (194.4, 90.0)
Routing:
- net Net-(C21-Pad1): track 60.7 -> 61.4 mm
- net Net-(C22-Pad2): track 59.6 -> 60.3 mm
